Commit message: Caster wheel and right wheel joints

File: description/robot_core.xacro (robot description, xacro)
@@ -13,3 +13,63 @@
       <color rgba="0 0 0 1" />
     </material>
+    <link name="base link">
+    </link>
+    <joint name="chassis joint" type="fixed">
+      <parent link="base_link"/>
+      <child link="chassis"/>
+      <origin xyz="-0.1 0 0"/>
+    </joint>
+    <link name="chassis">
+      <visual>
+        <origin xyz="0.15 0 0 .075"/>
+        <geometry>
+          <box size="0.3 0.3 0.15"/>
+        </geometry>
+        <material name="white"/>
+      </visual>
+    </link>
+    <!-- LEFT WHEEL LINK -->
+    <joint name="left_wheel_joint" type="continuous">
+      <parent link="base_link"/>
+      <child link="left_wheel"/>
+      <origin xyz="0 0.175 0" rpy="-${pi/2} 0 0"/>
+      <axis xyz="0 0 1"/>
+    </joint>
+    <link name="left_wheel">
+      <visual>
+        <geometry>
+          <cylinder radius="0.05" length="0.04"/>
+        </geometry>
+        <material name="blue"/>
+      </visual>
+    </link>
+    <!-- RIGHT WHEEL LINK -->
+    <joint name="right_wheel_joint" type="continuous">
+      <parent link="base_link"/>
+      <child link="right_wheel"/>
+      <origin xyz="0 -0.175 0" rpy="${pi/2} 0 0"/>
+      <axis xyz="0 0 -1"/>
+    </joint>
+    <link name="right_wheel">
+      <visual>
+        <geometry>
+          <cylinder radius="0.05" length="0.04"/>
+        </geometry>
+        <material name="blue"/>
+      </visual>
+    </link>
+    <!-- CASTER WHEEL LINK -->
+    <joint name="caster_wheel_joint" type="fixed">
+      <parent link="chassis"/>
+      <child link="caster_wheel"/>
+      <origin xyz="0.24 0 0"/>
+    </joint>
+    <link name="caster_wheel">
+      <visual>
+        <geometry>
+          <sphere radius="0.05"/>
+        </geometry>
+        <material name="black"/>
+      </visual>
+    </link>
 </robot>

Commit message: Collisions

File: description/robot_core.xacro (robot description, xacro)
@@ -15,4 +15,5 @@
     <link name="base link">
     </link>
+    <!-- CHASSIS LINK -->
     <joint name="chassis joint" type="fixed">
       <parent link="base_link"/>
@@ -28,4 +29,10 @@
         <material name="white"/>
       </visual>
+      <collision>
+        <origin xyz="0.15 0 0 .075"/>
+        <geometry>
+          <box size="0.3 0.3 0.15"/>
+        </geometry>
+      </collision>
     </link>
     <!-- LEFT WHEEL LINK -->
@@ -43,4 +50,9 @@
         <material name="blue"/>
       </visual>
+      <collision>
+        <geometry>
+          <cylinder radius="0.05" length="0.04"/>
+        </geometry>
+      </collision>
     </link>
     <!-- RIGHT WHEEL LINK -->
@@ -58,4 +70,9 @@
         <material name="blue"/>
       </visual>
+      <collision>
+        <geometry>
+          <cylinder radius="0.05" length="0.04"/>
+        </geometry>
+      </collision>
     </link>
     <!-- CASTER WHEEL LINK -->
@@ -72,4 +89,9 @@
         <material name="black"/>
       </visual>
+      <collision>
+        <geometry>
+          <sphere radius="0.05"/>
+        </geometry>
+      </collision>
     </link>
 </robot>

Commit message: inertial macros

File: description/robot_core.xacro (robot description, xacro)
@@ -1,4 +1,5 @@
 <?xml version="1.0"?>
 <robot xmlns:xacro="http://www.ros.org/wiki/xacro"  name="robot">
+  <xacro:include filename="inertial_macros.xacro"/>
     <material name="white">
       <color rgba="1 1 1 1" />
@@ -35,4 +36,7 @@
         </geometry>
       </collision>
+      <xacro:inertial_box mass="0.5" x="0.3" y="0.3" z="0.15">
+        <origin xyz="0.15 0 0 0.075" rpy="0 0 0"/>
+      </xacro:inertial_box>
     </link>
     <!-- LEFT WHEEL LINK -->
@@ -55,4 +59,7 @@
         </geometry>
       </collision>
+      <xacro:inertial_cylinder mass="0.1" length="0.04" radius="0.05">
+            <origin xyz="0 0 0" rpy="0 0 0"/>
+      </xacro:inertial_cylinder>
     </link>
     <!-- RIGHT WHEEL LINK -->
@@ -75,4 +82,7 @@
         </geometry>
       </collision>
+      <xacro:inertial_cylinder mass="0.1" length="0.04" radius="0.05">
+            <origin xyz="0 0 0" rpy="0 0 0"/>
+        </xacro:inertial_cylinder>
     </link>
     <!-- CASTER WHEEL LINK -->
@@ -94,4 +104,7 @@
         </geometry>
       </collision>
+      <xacro:inertial_sphere mass="0.1" radius="0.05">
+            <origin xyz="0 0 0" rpy="0 0 0"/>
+        </xacro:inertial_sphere>
     </link>
 </robot>
