Commit message: Gazebo control

File: description/robot.urdf.xacro (robot description, xacro)
@@ -2,3 +2,4 @@
 <robot xmlns:xacro="http://www.ros.org/wiki/xacro" name="robot">
     <xacro:include filename="robot_core.xacro" />
+    <xacro:include filename="gazebo_control.xacro" />
 </robot>

File: description/robot_core.xacro (robot description, xacro)
@@ -66,4 +66,7 @@
     </xacro:inertial_cylinder>
   </link>
+  <gazebo reference="left_wheel">
+    <material>Gazebo/Blue</material>
+  </gazebo>
   <!-- RIGHT WHEEL LINK -->
   <joint name="right_wheel_joint" type="continuous">
@@ -89,4 +92,7 @@
     </xacro:inertial_cylinder>
   </link>
+  <gazebo reference="right_wheel">
+    <material>Gazebo/Blue</material>
+  </gazebo>
   <!-- CASTER WHEEL LINK -->
   <joint name="caster_wheel_joint" type="fixed">
@@ -111,3 +117,6 @@
     </xacro:inertial_sphere>
   </link>
+  <gazebo reference="chassis">
+    <material>Gazebo/Black</material>
+  </gazebo>
 </robot>

Commit message: Fix moving in ros2 for now?

File: description/robot.urdf.xacro (robot description, xacro)
@@ -2,4 +2,7 @@
 <robot xmlns:xacro="http://www.ros.org/wiki/xacro" name="robot">
     <xacro:include filename="robot_core.xacro" />
-    <xacro:include filename="gazebo_control.xacro" />
+    <!-- <xacro:include filename="ros2_control.xacro" /> -->
+    <xacro:include filename="gazebo_control_copy.xacro" />
+    <xacro:include filename="lidar.xacro" />
+    <!-- <xacro:include filename="gazebo_control.xacro" /> -->
 </robot>

File: description/robot_core.xacro (robot description, xacro)
@@ -1,5 +1,5 @@
 <?xml version="1.0"?>
 <robot xmlns:xacro="http://www.ros.org/wiki/xacro" name="robot">
-  <xacro:include filename="$(dirname)/inertial_macros.xacro" />
+<xacro:include filename="$(find my_bot)/description/inertial_macros.xacro" />
   <material name="white">
     <color rgba="1 1 1 1" />
@@ -14,5 +14,5 @@
     <color rgba="0 0 0 1" />
   </material>
-  <link name="base link">
+  <link name="base_link">
   </link>
   <!-- CHASSIS LINK -->
@@ -24,5 +24,5 @@
   <link name="chassis">
     <visual>
-      <origin xyz="0.15 0 0 .075" />
+      <origin xyz="0.15 0 0.075" />
       <geometry>
         <box size="0.3 0.3 0.15" />
@@ -31,5 +31,5 @@
     </visual>
     <collision>
-      <origin xyz="0.15 0 0 .075" />
+      <origin xyz="0.15 0 0.075" />
       <geometry>
         <box size="0.3 0.3 0.15" />
@@ -37,5 +37,5 @@
     </collision>
     <xacro:inertial_box mass="0.5" x="0.3" y="0.3" z="0.15">
-      <origin xyz="0.15 0 0 0.075" rpy="0 0 0" />
+      <origin xyz="0.15 0 0.075" rpy="0 0 0" />
     </xacro:inertial_box>
   </link>
@@ -117,8 +117,8 @@
     </xacro:inertial_sphere>
   </link>
-  <gazebo reference="chassis">
-    <material>Gazebo/Black</material>
-    <mul1 value="000.1" />
-    <mul2 value="000.1" />
-  </gazebo>
+  <gazebo reference="caster_wheel">
+  <material>Gazebo/Black</material>
+  <mu1>0.001</mu1>
+  <mu2>0.001</mu2>
+</gazebo>
 </robot>
